File: 1BIT_ATTENUATOR_CH_A.kicad_sch (KiCad schematic)
At the start: 9 parts, among them IC36 ${DEVICE}, IC37 ${DEVICE}, IC38 ${DEVICE}

Commit message: Rerouted PCB Logic part
Parts:
- renumbered C111 to C901, C112 to C902, C113 to C903, C114 to C904, IC36 to IC901, IC37 to IC902, IC38 to IC903, R79 to R901, R80 to R902
Changed lines of the file:
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@@
 		(dnp no)
 		(fields_autoplaced yes)
-		(property "Reference" "C111"
+		(property "Reference" "C901"
 			(at 88.9 102.87 0)
 			(effects
@@
 			(project "8CH_Analog_Front_END"
 				(path "/41597329-5145-432a-9041-5bc2cec82d9b/e0337a1b-c397-4f99-b607-786eab07764a/b9931bc0-163e-4a03-a053-c84ed198459e"
-					(reference "C111")
+					(reference "C901")
 					(unit 1)
 				)
@@
 		(dnp no)
 		(fields_autoplaced yes)
-		(property "Reference" "R80"
+		(property "Reference" "R902"
 			(at 358.14 114.9349 90)
 			(effects
@@
 			(project "8CH_Analog_Front_END"
 				(path "/41597329-5145-432a-9041-5bc2cec82d9b/e0337a1b-c397-4f99-b607-786eab07764a/b9931bc0-163e-4a03-a053-c84ed198459e"
-					(reference "R80")
+					(reference "R902")
 					(unit 1)
 				)
@@
 		(dnp no)
 		(fields_autoplaced yes)
-		(property "Reference" "#PWR0193"
+		(property "Reference" "#PWR0908"
 			(at 355.6 129.54 0)
 			(effects
@@
 			(project "8CH_Analog_Front_END"
 				(path "/41597329-5145-432a-9041-5bc2cec82d9b/e0337a1b-c397-4f99-b607-786eab07764a/b9931bc0-163e-4a03-a053-c84ed198459e"
-					(reference "#PWR0193")
+					(reference "#PWR0908")
 					(unit 1)
 				)
@@
 		(dnp no)
 		(fields_autoplaced yes)
-		(property "Reference" "IC36"
+		(property "Reference" "IC901"
 			(at 128.27 91.44 0)
 			(effects
@@
 			(project "8CH_Analog_Front_END"
 				(path "/41597329-5145-432a-9041-5bc2cec82d9b/e0337a1b-c397-4f99-b607-786eab07764a/b9931bc0-163e-4a03-a053-c84ed198459e"
-					(reference "IC36")
+					(reference "IC901")
 					(unit 1)
 				)
@@
 		(dnp no)
 		(fields_autoplaced yes)
-		(property "Reference" "IC37"
+		(property "Reference" "IC902"
 			(at 207.01 101.6 0)
 			(effects
@@
 			(project "8CH_Analog_Front_END"
 				(path "/41597329-5145-432a-9041-5bc2cec82d9b/e0337a1b-c397-4f99-b607-786eab07764a/b9931bc0-163e-4a03-a053-c84ed198459e"
-					(reference "IC37")
+					(reference "IC902")
 					(unit 1)
 				)
@@
 		(dnp no)
 		(fields_autoplaced yes)
-		(property "Reference" "C113"
+		(property "Reference" "C903"
 			(at 246.38 102.87 0)
 			(effects
@@
 			(project "8CH_Analog_Front_END"
 				(path "/41597329-5145-432a-9041-5bc2cec82d9b/e0337a1b-c397-4f99-b607-786eab07764a/b9931bc0-163e-4a03-a053-c84ed198459e"
-					(reference "C113")
+					(reference "C903")
 					(unit 1)
 				)
@@
 		(dnp no)
 		(fields_autoplaced yes)
-		(property "Reference" "#PWR0187"
+		(property "Reference" "#PWR0905"
 			(at 217.17 123.19 0)
 			(effects
@@
 			(project "8CH_Analog_Front_END"
 				(path "/41597329-5145-432a-9041-5bc2cec82d9b/e0337a1b-c397-4f99-b607-786eab07764a/b9931bc0-163e-4a03-a053-c84ed198459e"
-					(reference "#PWR0187")
+					(reference "#PWR0905")
 					(unit 1)
 				)
@@
 		(dnp no)
 		(fields_autoplaced yes)
-		(property "Reference" "#PWR0190"
+		(property "Reference" "#PWR0901"
 			(at 58.42 129.54 0)
 			(effects
@@
 			(project "8CH_Analog_Front_END"
 				(path "/41597329-5145-432a-9041-5bc2cec82d9b/e0337a1b-c397-4f99-b607-786eab07764a/b9931bc0-163e-4a03-a053-c84ed198459e"
-					(reference "#PWR0190")
+					(reference "#PWR0901")
 					(unit 1)
 				)
@@
 		(dnp no)
 		(fields_autoplaced yes)
-		(property "Reference" "IC38"
+		(property "Reference" "IC903"
 			(at 285.75 111.76 0)
 			(effects
@@
 			(project "8CH_Analog_Front_END"
 				(path "/41597329-5145-432a-9041-5bc2cec82d9b/e0337a1b-c397-4f99-b607-786eab07764a/b9931bc0-163e-4a03-a053-c84ed198459e"
-					(reference "IC38")
+					(reference "IC903")
 					(unit 1)
 				)
@@
 		(dnp no)
 		(fields_autoplaced yes)
-		(property "Reference" "#PWR0189"
+		(property "Reference" "#PWR0902"
 			(at 113.03 130.81 0)
 			(effects
@@
 			(project "8CH_Analog_Front_END"
 				(path "/41597329-5145-432a-9041-5bc2cec82d9b/e0337a1b-c397-4f99-b607-786eab07764a/b9931bc0-163e-4a03-a053-c84ed198459e"
-					(reference "#PWR0189")
+					(reference "#PWR0902")
 					(unit 1)
 				)
@@
 		(dnp no)
 		(fields_autoplaced yes)
-		(property "Reference" "#PWR0188"
+		(property "Reference" "#PWR0906"
 			(at 270.51 72.39 0)
 			(effects
@@
 			(project "8CH_Analog_Front_END"
 				(path "/41597329-5145-432a-9041-5bc2cec82d9b/e0337a1b-c397-4f99-b607-786eab07764a/b9931bc0-163e-4a03-a053-c84ed198459e"
-					(reference "#PWR0188")
+					(reference "#PWR0906")
 					(unit 1)
 				)
@@
 		(dnp no)
 		(fields_autoplaced yes)
-		(property "Reference" "#PWR0192"
+		(property "Reference" "#PWR0907"
 			(at 300.99 72.39 0)
 			(effects
@@
 			(project "8CH_Analog_Front_END"
 				(path "/41597329-5145-432a-9041-5bc2cec82d9b/e0337a1b-c397-4f99-b607-786eab07764a/b9931bc0-163e-4a03-a053-c84ed198459e"
-					(reference "#PWR0192")
+					(reference "#PWR0907")
 					(unit 1)
 				)
@@
 		(dnp no)
 		(fields_autoplaced yes)
-		(property "Reference" "#PWR0191"
+		(property "Reference" "#PWR0903"
 			(at 143.51 130.81 0)
 			(effects
@@
 			(project "8CH_Analog_Front_END"
 				(path "/41597329-5145-432a-9041-5bc2cec82d9b/e0337a1b-c397-4f99-b607-786eab07764a/b9931bc0-163e-4a03-a053-c84ed198459e"
-					(reference "#PWR0191")
+					(reference "#PWR0903")
 					(unit 1)
 				)
@@
 		(dnp no)
 		(fields_autoplaced yes)
-		(property "Reference" "#PWR0186"
+		(property "Reference" "#PWR0904"
 			(at 196.85 123.19 0)
 			(effects
@@
 			(project "8CH_Analog_Front_END"
 				(path "/41597329-5145-432a-9041-5bc2cec82d9b/e0337a1b-c397-4f99-b607-786eab07764a/b9931bc0-163e-4a03-a053-c84ed198459e"
-					(reference "#PWR0186")
+					(reference "#PWR0904")
 					(unit 1)
 				)
@@
 		(dnp no)
 		(fields_autoplaced yes)
-		(property "Reference" "C114"
+		(property "Reference" "C904"
 			(at 325.12 102.87 0)
 			(effects
@@
 			(project "8CH_Analog_Front_END"
 				(path "/41597329-5145-432a-9041-5bc2cec82d9b/e0337a1b-c397-4f99-b607-786eab07764a/b9931bc0-163e-4a03-a053-c84ed198459e"
-					(reference "C114")
+					(reference "C904")
 					(unit 1)
 				)
@@
 		(dnp no)
 		(fields_autoplaced yes)
-		(property "Reference" "R79"
+		(property "Reference" "R901"
 			(at 60.96 114.9349 90)
 			(effects
@@
 			(project "8CH_Analog_Front_END"
 				(path "/41597329-5145-432a-9041-5bc2cec82d9b/e0337a1b-c397-4f99-b607-786eab07764a/b9931bc0-163e-4a03-a053-c84ed198459e"
-					(reference "R79")
+					(reference "R901")
 					(unit 1)
 				)
@@
 		(dnp no)
 		(fields_autoplaced yes)
-		(property "Reference" "C112"
+		(property "Reference" "C902"
 			(at 167.64 102.87 0)
 			(effects
@@
 			(project "8CH_Analog_Front_END"
 				(path "/41597329-5145-432a-9041-5bc2cec82d9b/e0337a1b-c397-4f99-b607-786eab07764a/b9931bc0-163e-4a03-a053-c84ed198459e"
-					(reference "C112")
+					(reference "C902")
 					(unit 1)
 				)
