File: 4BIT_STEP_ATTENUATOR_CH_A.kicad_sch (KiCad schematic)
At the start: 7 parts, among them IC701 ${DEVICE}

Commit message: Rerouted PCB Logic part
Parts:
- renumbered C704 to C703, C703 to C704, L702 to L701, L701 to L702
Changed lines of the file:
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@@
 		(dnp no)
 		(fields_autoplaced yes)
-		(property "Reference" "#PWR0705"
+		(property "Reference" "#PWR0702"
 			(at 180.34 130.81 0)
 			(effects
@@
 			(project "8CH_Analog_Front_END"
 				(path "/41597329-5145-432a-9041-5bc2cec82d9b/e0337a1b-c397-4f99-b607-786eab07764a/40227e70-2d37-4426-8ded-7de7d9cfeb10"
-					(reference "#PWR0705")
+					(reference "#PWR0702")
 					(unit 1)
 				)
@@
 		(dnp no)
 		(fields_autoplaced yes)
-		(property "Reference" "C703"
+		(property "Reference" "C704"
 			(at 201.93 99.0599 90)
 			(effects
@@
 			(project "8CH_Analog_Front_END"
 				(path "/41597329-5145-432a-9041-5bc2cec82d9b/e0337a1b-c397-4f99-b607-786eab07764a/40227e70-2d37-4426-8ded-7de7d9cfeb10"
-					(reference "C703")
+					(reference "C704")
 					(unit 1)
 				)
@@
 		(dnp no)
 		(fields_autoplaced yes)
-		(property "Reference" "#PWR0703"
+		(property "Reference" "#PWR0701"
 			(at 137.16 130.81 0)
 			(effects
@@
 			(project "8CH_Analog_Front_END"
 				(path "/41597329-5145-432a-9041-5bc2cec82d9b/e0337a1b-c397-4f99-b607-786eab07764a/40227e70-2d37-4426-8ded-7de7d9cfeb10"
-					(reference "#PWR0703")
+					(reference "#PWR0701")
 					(unit 1)
 				)
@@
 		(on_board yes)
 		(dnp no)
-		(property "Reference" "#PWR0701"
+		(property "Reference" "#PWR0703"
 			(at 186.69 105.41 0)
 			(effects
@@
 			(project "8CH_Analog_Front_END"
 				(path "/41597329-5145-432a-9041-5bc2cec82d9b/e0337a1b-c397-4f99-b607-786eab07764a/40227e70-2d37-4426-8ded-7de7d9cfeb10"
-					(reference "#PWR0701")
+					(reference "#PWR0703")
 					(unit 1)
 				)
@@
 		(on_board yes)
 		(dnp no)
-		(property "Reference" "L701"
+		(property "Reference" "L702"
 			(at 211.582 101.6 0)
 			(effects
@@
 			(project "8CH_Analog_Front_END"
 				(path "/41597329-5145-432a-9041-5bc2cec82d9b/e0337a1b-c397-4f99-b607-786eab07764a/40227e70-2d37-4426-8ded-7de7d9cfeb10"
-					(reference "L701")
+					(reference "L702")
 					(unit 1)
 				)
@@
 		(dnp no)
 		(fields_autoplaced yes)
-		(property "Reference" "#PWR0702"
+		(property "Reference" "#PWR0704"
 			(at 198.12 113.03 0)
 			(effects
@@
 			(project "8CH_Analog_Front_END"
 				(path "/41597329-5145-432a-9041-5bc2cec82d9b/e0337a1b-c397-4f99-b607-786eab07764a/40227e70-2d37-4426-8ded-7de7d9cfeb10"
-					(reference "#PWR0702")
+					(reference "#PWR0704")
 					(unit 1)
 				)
@@
 		(dnp no)
 		(fields_autoplaced yes)
-		(property "Reference" "C704"
+		(property "Reference" "C703"
 			(at 184.15 116.8399 90)
 			(effects
@@
 			(project "8CH_Analog_Front_END"
 				(path "/41597329-5145-432a-9041-5bc2cec82d9b/e0337a1b-c397-4f99-b607-786eab07764a/40227e70-2d37-4426-8ded-7de7d9cfeb10"
-					(reference "C704")
+					(reference "C703")
 					(unit 1)
 				)
@@
 		(dnp no)
 		(fields_autoplaced yes)
-		(property "Reference" "#PWR0704"
+		(property "Reference" "#PWR0705"
 			(at 213.36 109.22 0)
 			(effects
@@
 			(project "8CH_Analog_Front_END"
 				(path "/41597329-5145-432a-9041-5bc2cec82d9b/e0337a1b-c397-4f99-b607-786eab07764a/40227e70-2d37-4426-8ded-7de7d9cfeb10"
-					(reference "#PWR0704")
+					(reference "#PWR0705")
 					(unit 1)
 				)
@@
 		(on_board yes)
 		(dnp no)
-		(property "Reference" "L702"
+		(property "Reference" "L701"
 			(at 184.912 106.68 0)
 			(effects
@@
 			(project "8CH_Analog_Front_END"
 				(path "/41597329-5145-432a-9041-5bc2cec82d9b/e0337a1b-c397-4f99-b607-786eab07764a/40227e70-2d37-4426-8ded-7de7d9cfeb10"
-					(reference "L702")
+					(reference "L701")
 					(unit 1)
 				)
