File: 4BIT_STEP_ATTENUATOR_CH_A.kicad_sch (KiCad schematic)
At the start: 7 parts, among them IC701 ${DEVICE}

Commit message: WIP snapshot
Parts:
- removed C701, C702: 10nF, Capacitors SMD:CAPC1005X55N, symbol CERN:Capacitors SMD/CC0402_10NF_50V_5%_X7R
- added C701, C702, C704, C706: 100nF, Capacitors SMD:CAPC1005X55N, symbol CERN:Capacitors SMD/CC0402_100NF_50V_10%_X7R
- added C707, C708, C714, C717: 10uF, Capacitors SMD:CAPC3216X180N, symbol CERN:Capacitors SMD/CC1206_10UF_50V_10%_X5R
- added C709, C710, C711, C712, C713, C715, C716: 100nF, Capacitors SMD:CAPC1608X87N, symbol CERN:Capacitors SMD/CC0603_100NF_50V_10%_X5R
- added IC702: ${DEVICE}, ICs And Semiconductors SMD:SOIC127P600X175-16N, symbol CERN:Analog & Interface/MAATCC0008
- added IC703: ${DEVICE}, ICs And Semiconductors SMD:SOT95P280X90-5N, symbol CERN:Regulators/ADP7182AUJZ-5.0-R7
- added IC704: ${DEVICE}, ICs And Semiconductors SMD:SOT127P700X180-6N, symbol CERN:Regulators/TPS7A4501DCQ
- added L702, L704: 220R@100MHz, Inductors SMD:INDC1608X95N, symbol CERN:Inductors SMD/IND0603_MURATA_BLM18SG221TN1 [alt]
- added L705, L706: 60R@100MHz, Inductors SMD:INDC4516X180N, symbol CERN:Inductors SMD/IND1806_MURATA_BLM41PG600SN1L [alt]
- added LD701, LD702: ${COLOR}, ICs And Semiconductors SMD:LED_KINGBRIGHT_KPH-1608CGCK, symbol CERN:LEDs & Displays/LED_KINGBRIGHT_KPH-1608CGCK
- added R701: 12k, Resistor_SMD:R_0603_1608Metric_Pad0.98x0.95mm_HandSolder, symbol Device:R
- added R702: 820, Resistor_SMD:R_0603_1608Metric_Pad0.98x0.95mm_HandSolder, symbol Device:R
- added R703: 4020, Resistor_SMD:R_0603_1608Metric_Pad0.98x0.95mm_HandSolder, symbol Device:R
- added R704: 510, Resistors SMD:RESC1608X55N, symbol CERN:Resistors SMD/R0603_510R_1%_0.1W_100PPM
- added R705: 510, Resistor_SMD:R_0603_1608Metric_Pad0.98x0.95mm_HandSolder, symbol Device:R
- renumbered C704 to C705, L702 to L703
Connections:
- net +5VA: now also C715.2, C716.2, C717.2, IC704.4 (OUT), L702.1, R701.2, R705.2
- net -5VA: now also C712.2, C713.2, C714.2, IC703.5 (VOUT), L704.2, R704.2
- net DIGITAL_STEP_ATT_IN_CH_A: now also C701.1
- net DIGITAL_STEP_ATT_OUT_CH_A: now also IC701.15 (RF2)
- net GND: now also C704.1, C706.1, C707.1, C708.1, C709.1, C710.1, C711.1, C712.1, C713.1, C714.1, C715.1, C716.1, C717.1, IC702.1 (GND), IC702.11 (GND), IC702.12 (GND), IC702.14 (GND), IC702.16 (GND), IC702.3 (GND), IC703.1 (GND), IC704.3 (GND), IC704.6 (GND), LD701.2 (A), LD702.1 (C), R703.1
- net at IC701.2 (RF1): now also C701.2
- new net: C708.2, C710.2, IC703.2 (VIN), IC703.3 (EN), L706.1
- new net: C702.2, IC702.2 (RF1)
- new net: C706.2, IC702.5 (VEE), L704.1
- new net: C704.2, IC702.6 (VCC), L702.2
- new net: LD702.2 (A), R705.1
- new net: C707.2, C709.2, C711.2, IC704.1 (~{SHDN}), IC704.2 (IN), L705.1
- new net: LD701.1 (C), R704.1
- new net: IC704.5 (ADJ), R702.1, R703.2
- new net: R701.1, R702.2
- new net +5V: L705.2
- new net -5V: L706.2
- new net C1_1dB_B: IC702.10 (C1)
- new net C2_2dB_B: IC702.9 (C2)
- new net C4_4dB_B: IC702.8 (C3)
- new net C8_8dB_B: IC702.7 (C4)
- new net DIGITAL_STEP_ATT_IN_CH_B: C702.1
- new net DIGITAL_STEP_ATT_OUT_CH_B: IC702.15 (RF2)
- no-connect marks 2 -> 5
Other:
- note added: "-5V"
- note added: "5V"

Commit message: Update project files and backups
Parts:
- removed R701: 12k, Resistor_SMD:R_0603_1608Metric_Pad0.98x0.95mm_HandSolder, symbol Device:R
- removed R702: 820, Resistor_SMD:R_0603_1608Metric_Pad0.98x0.95mm_HandSolder, symbol Device:R
- removed R703: 4020, Resistor_SMD:R_0603_1608Metric_Pad0.98x0.95mm_HandSolder, symbol Device:R
- removed R705: 510, Resistor_SMD:R_0603_1608Metric_Pad0.98x0.95mm_HandSolder, symbol Device:R
- added R701, R703: 4k7, Resistors SMD:RESC1608X55N, symbol CERN:Resistors SMD/R0603_4K7_1%_0.1W_100PPM
- added R702: 10k, Resistors SMD:RESC1608X55N, symbol CERN:Resistors SMD/R0603_10K_1%_0.1W_100PPM
- added R706: 510, Resistors SMD:RESC1608X55N, symbol CERN:Resistors SMD/R0603_510R_1%_0.1W_100PPM
Connections:
- net +5VA: now also R701.1, R706.2
- net GND: now also R703.2
- net at LD702.2 (A): now also R706.1
- net at IC704.5 (ADJ): now also R702.1, R703.1
- new net: R701.2, R702.2
Other:
- note added: "R1 = 14k7 R2 = 4k7 VOut = 4.99V"
