File: AFE_BLOCK.kicad_sch (KiCad schematic)
At the start: 3 parts, among them U1 LPF, U2 LPF

Commit message: Updated schematic and rerouted PCB
Parts:
- removed FTG1: Use only in PCB, Pads:FIDUCIAL_TOP_C100-200, symbol CERN:Pads/FIDUCIAL_TARGET_C100-200

Commit message: Rerouted PCB Logic part
Parts:
- renumbered U1 to U501, U2 to U502
Changed lines of the file:
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@@
 		(dnp no)
 		(fields_autoplaced yes)
-		(property "Reference" "#PWR0163"
+		(property "Reference" "#PWR0502"
 			(at 59.69 140.97 0)
 			(effects
@@
 			(project ""
 				(path "/41597329-5145-432a-9041-5bc2cec82d9b/e0337a1b-c397-4f99-b607-786eab07764a"
-					(reference "#PWR0163")
+					(reference "#PWR0502")
 					(unit 1)
 				)
@@
 		(dnp no)
 		(fields_autoplaced yes)
-		(property "Reference" "#PWR0165"
+		(property "Reference" "#PWR0501"
 			(at 59.69 113.03 0)
 			(effects
@@
 			(project ""
 				(path "/41597329-5145-432a-9041-5bc2cec82d9b/e0337a1b-c397-4f99-b607-786eab07764a"
-					(reference "#PWR0165")
+					(reference "#PWR0501")
 					(unit 1)
 				)
@@
 		(dnp no)
 		(fields_autoplaced yes)
-		(property "Reference" "U2"
+		(property "Reference" "U502"
 			(at 45.085 111.76 0)
 			(effects
@@
 			(project ""
 				(path "/41597329-5145-432a-9041-5bc2cec82d9b/e0337a1b-c397-4f99-b607-786eab07764a"
-					(reference "U2")
+					(reference "U502")
 					(unit 1)
 				)
@@
 		(dnp no)
 		(fields_autoplaced yes)
-		(property "Reference" "U1"
+		(property "Reference" "U501"
 			(at 45.085 83.82 0)
 			(effects
@@
 			(project ""
 				(path "/41597329-5145-432a-9041-5bc2cec82d9b/e0337a1b-c397-4f99-b607-786eab07764a"
-					(reference "U1")
-					(unit 1)
-				)
+					(reference "U501")
+					(unit 1)
+				)
