File: AFE_BLOCK.kicad_sch (KiCad schematic)
At the start: 2 parts, among them U501 LPF, U502 LPF

Commit message: WIP snapshot
Other:
- removed sheet 4BIT_STEP_ATTENUATOR_CH_B
- sheet 1BIT_ATTENUATOR_CH_B: file 1BIT_ATTENUATOR_CH_B.kicad_sch -> 1BIT_ATTENUATOR_CH_A.kicad_sch
- sheet 1BIT_ATTENUATOR_CH_B ports: added 1BIT_ATTEN_VC1_CH_A, 1BIT_ATTEN_VC2_CH_A, 1_BIT_ATT_IN_CH_A; removed 1BIT_ATTEN_VC1_CH_B, 1BIT_ATTEN_VC2_CH_B, 1_BIT_ATT_IN_CH_B
- sheet 4BIT_STEP_ATTENUATOR_CH_A ports: added C1_1dB_B, C2_2dB_B, C4_4dB_B, C8_8dB_B, DIGITAL_STEP_ATT_IN_CH_B, DIGITAL_STEP_ATT_OUT_CH_B; removed none
- sheet LOGIC_CONTROL_CH_A: file LOGIC_CONTROL_CH_A.kicad_sch -> CHANNEL_LOGIC_CONTROL.kicad_sch
- sheet LOGIC_CONTROL_CH_A ports: added 1BITTTEN_VC1_CH, 1BITTTEN_VC2_CH, C1_1dB, C2_2dB, C4_4dB, C8_8dB, CAL_MEAS_SW_VC1_CH, CAL_MEAS_SW_VC2_CH, DAC_DIR_V1_CH, DAC_DIR_V2_CH, OPAMP_BYPASS_V1_CH, OPAMP_BYPASS_V2_CH, SER_DATA_IN, SER_RCLK, SER_RST_N; removed 1BIT_ATTEN_VC1_CH_A, 1BIT_ATTEN_VC2_CH_A, C1_1dB_A, C2_2dB_A, C4_4dB_A, C8_8dB_A, CAL_MEAS_SW_VC1_CH_A, CAL_MEAS_SW_VC2_CH_A, DAC_DIR_V1_CH_A, DAC_DIR_V2_CH_A, D_LATCH_OE, OPAMP_BYPASS_V1_CH_A, OPAMP_BYPASS_V2_CH_A, SER_DATA, SER_LATCH_CH_A
- sheet LOGIC_CONTROL_CH_B: file LOGIC_CONTROL_CH_B.kicad_sch -> CHANNEL_LOGIC_CONTROL.kicad_sch
- sheet LOGIC_CONTROL_CH_B ports: added 1BITTTEN_VC1_CH, 1BITTTEN_VC2_CH, A0, A1, A2, A3, A4, A5, A6, C1_1dB, C2_2dB, C4_4dB, C8_8dB, CAL_MEAS_SW_VC1_CH, CAL_MEAS_SW_VC2_CH, DAC_DIR_V1_CH, DAC_DIR_V2_CH, OPAMP_BYPASS_V1_CH, OPAMP_BYPASS_V2_CH, SER_DATA_IN, SER_RCLK, SER_RST_N; removed 1BIT_ATTEN_VC1_CH_B, 1BIT_ATTEN_VC2_CH_B, B0, B1, B2, B3, B4, B5, B6, C1_1dB_B, C2_2dB_B, C4_4dB_B, C8_8dB_B, CAL_MEAS_SW_VC1_CH_B, CAL_MEAS_SW_VC2_CH_B, DAC_DIR_V1_CH_B, DAC_DIR_V2_CH_B, D_LATCH_OE, OPAMP_BYPASS_V1_CH_B, OPAMP_BYPASS_V2_CH_B, SER_DATA, SER_LATCH_CH_B

Commit message: Update project files and backups
Parts:
- added R501: 10k, Resistors SMD:RESC1005X40N, symbol CERN:Resistors SMD/R0402_10K_1%_0.0625W_100PPM
Connections:
- net SER_RST_N: now also R501.1
- new net +3V3D: R501.2
- no-connect marks 2 -> 5
Other:
- sheet LOGIC_CONTROL_CH_A ports: added IO_3V3_0, IO_3V3_1, IO_3V3_2, IO_3V3_3, IO_3V3_4, IO_3V3_5, IO_3V3_6, IO_5V_0, IO_5V_1, IO_5V_10, IO_5V_11, IO_5V_12, IO_5V_13, IO_5V_14, IO_5V_15, IO_5V_2, IO_5V_3, IO_5V_4, IO_5V_5, IO_5V_6, IO_5V_7, IO_5V_8, IO_5V_9; removed 1BITTTEN_VC1_CH, 1BITTTEN_VC2_CH, A0, A1, A2, A3, A4, A5, A6, C1_1dB, C2_2dB, C4_4dB, C8_8dB, CAL_MEAS_SW_VC1_CH, CAL_MEAS_SW_VC2_CH, DAC_DIR_V1_CH, DAC_DIR_V2_CH, OPAMP_BYPASS_V1_CH, OPAMP_BYPASS_V2_CH
- sheet LOGIC_CONTROL_CH_B ports: added IO_3V3_0, IO_3V3_1, IO_3V3_2, IO_3V3_3, IO_3V3_4, IO_3V3_5, IO_3V3_6, IO_5V_0, IO_5V_1, IO_5V_10, IO_5V_11, IO_5V_12, IO_5V_13, IO_5V_14, IO_5V_15, IO_5V_2, IO_5V_3, IO_5V_4, IO_5V_5, IO_5V_6, IO_5V_7, IO_5V_8, IO_5V_9; removed 1BITTTEN_VC1_CH, 1BITTTEN_VC2_CH, A0, A1, A2, A3, A4, A5, A6, C1_1dB, C2_2dB, C4_4dB, C8_8dB, CAL_MEAS_SW_VC1_CH, CAL_MEAS_SW_VC2_CH, DAC_DIR_V1_CH, DAC_DIR_V2_CH, OPAMP_BYPASS_V1_CH, OPAMP_BYPASS_V2_CH
- note added: "Swap pins at your convenience (making sure 3.3V pins are not mixed with 5V pins). RF blocking caps next to pins of relevant control inputs, on top layer. Example: IC1606, IC1706 on layout."
