File: DAC_AMPLIFIER_CH_A.kicad_sch (KiCad schematic)
At the start: 26 parts, among them IC47 ${DEVICE}, IC48 ${DEVICE}, IC49 ${DEVICE}

Commit message: Updated schematic and rerouted PCB
Connections:
- net OPAMP_BYPASS_V1_CH_A: now also IC47.4 (V2); no longer IC47.6 (V1)
- net OPAMP_BYPASS_V2_CH_A: now also IC47.6 (V1); no longer IC47.4 (V2)
- net at C135.1: now also IC47.1 (RF1); no longer IC47.3 (RF2)
- net at C134.1, R83.2: now also IC47.3 (RF2); no longer IC47.1 (RF1)
Other:
- moved on the sheet: IC47
Changed lines of the file:
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@@
 	(wire
 		(pts
-			(xy 114.3 116.84) (xy 114.3 120.65)
+			(xy 110.49 88.9) (xy 110.49 92.71)
 		)
 		(stroke
@@
 	(wire
 		(pts
-			(xy 116.84 116.84) (xy 114.3 116.84)
+			(xy 110.49 88.9) (xy 116.84 88.9)
 		)
 		(stroke
@@
 	(wire
 		(pts
+			(xy 116.84 88.9) (xy 116.84 96.52)
+		)
+		(stroke
+			(width 0)
+			(type default)
+		)
+	)
+	(wire
+		(pts
 			(xy 289.56 101.6) (xy 293.37 101.6)
 		)
@@
 	(symbol
 		(lib_id "CERN:Analog & Interface/MASW-008853")
-		(at 121.92 99.06 0)
+		(at 121.92 114.3 0)
+		(mirror x)
 		(unit 1)
 		(exclude_from_sim no)
@@
 		(on_board yes)
 		(dnp no)
-		(fields_autoplaced yes)
 		(property "Reference" "IC47"
-			(at 129.54 93.98 0)
+			(at 129.54 119.38 0)
 			(effects
 				(font
@@
 		)
 		(property "Value" "${DEVICE}"
-			(at 129.54 96.52 0)
+			(at 129.54 116.84 0)
 			(effects
 				(font
@@
 		)
 		(property "Footprint" "ICs And Semiconductors SMD:SOT65P210X110-6N"
-			(at 121.92 99.06 0)
+			(at 121.92 114.3 0)
 			(effects
 				(font
@@
 		)
 		(property "Datasheet" "${CERN_DATASHEET_DIR}\\MASW-008853.pdf"
-			(at 121.92 99.06 0)
+			(at 121.92 114.3 0)
 			(effects
 				(font
@@
 		)
 		(property "Description" "GaAs SPDT 2.7 V High Power Switch DC - 5.0 GHz"
-			(at 121.92 99.06 0)
+			(at 121.92 114.3 0)
 			(effects
 				(font
@@
 		)
 		(property "Manufacturer" "MACOM"
-			(at 121.92 99.06 0)
+			(at 121.92 114.3 0)
 			(show_name yes)
 			(effects
@@
 		)
 		(property "Comment" "MASW-008853"
-			(at 121.92 99.06 0)
+			(at 121.92 114.3 0)
 			(show_name yes)
 			(effects
@@
 		)
 		(property "Component Kind" "Standard"
-			(at 121.92 99.06 0)
+			(at 121.92 114.3 0)
 			(show_name yes)
 			(effects
@@
 		)
 		(property "Component Type" "Standard"
-			(at 121.92 99.06 0)
+			(at 121.92 114.3 0)
 			(show_name yes)
 			(effects
@@
 		)
 		(property "Device" "MASW-008853"
-			(at 121.92 99.06 0)
+			(at 121.92 114.3 0)
 			(show_name yes)
 			(effects
@@
 		)
 		(property "PackageDescription" "SOT363, SC70-6, 0.65mm Pitch; 6 pin, 1.25mm W X 2.00mm L X 1.10mm H body, IPC Medium Density"
-			(at 121.92 99.06 0)
+			(at 121.92 114.3 0)
 			(show_name yes)
 			(effects
@@
 		)
 		(property "Status" ""
-			(at 121.92 99.06 0)
+			(at 121.92 114.3 0)
 			(show_name yes)
 			(effects
@@
 		)
 		(property "Part Description" "GaAs SPDT 2.7 V High Power Switch DC - 5.0 GHz"
-			(at 121.92 99.06 0)
+			(at 121.92 114.3 0)
 			(show_name yes)
 			(effects
@@
 		)
 		(property "Manufacturer Part Number" "MASW-008853"
-			(at 121.92 99.06 0)
+			(at 121.92 114.3 0)
 			(show_name yes)
 			(effects
@@
 		)
 		(property "Pin Count" "6"
-			(at 121.92 99.06 0)
+			(at 121.92 114.3 0)
 			(show_name yes)
 			(effects
@@
 		)
 		(property "Case" "SOT363"
-			(at 121.92 99.06 0)
+			(at 121.92 114.3 0)
 			(show_name yes)
 			(effects
@@
 		)
 		(property "Mounted" "Yes"
-			(at 121.92 99.06 0)
+			(at 121.92 114.3 0)
 			(show_name yes)
 			(effects
@@
 		)
 		(property "Socket" "No"
-			(at 121.92 99.06 0)
+			(at 121.92 114.3 0)
 			(show_name yes)
 			(effects
@@
 		)
 		(property "SMD" "Yes"
-			(at 121.92 99.06 0)
+			(at 121.92 114.3 0)
 			(show_name yes)
 			(effects
@@
 		)
 		(property "PressFit" "No"
-			(at 121.92 99.06 0)
+			(at 121.92 114.3 0)
 			(show_name yes)
 			(effects
@@
 		)
 		(property "Sense" "No"
-			(at 121.92 99.06 0)
+			(at 121.92 114.3 0)
 			(show_name yes)
 			(effects
@@
 		)
 		(property "Sense Comment" ""
-			(at 121.92 99.06 0)
+			(at 121.92 114.3 0)
 			(show_name yes)
 			(effects
@@
 		)
 		(property "Bonding" "No"
-			(at 121.92 99.06 0)
+			(at 121.92 114.3 0)
 			(show_name yes)
 			(effects
@@
 		)
 		(property "Status Comment" ""
-			(at 121.92 99.06 0)
+			(at 121.92 114.3 0)
 			(show_name yes)
 			(effects
@@
 		)
 		(property "ComponentHeight" "1.1mm"
-			(at 121.92 99.06 0)
+			(at 121.92 114.3 0)
 			(show_name yes)
 			(effects
@@
 		)
 		(property "Author" "CERN DEM HF"
-			(at 121.92 99.06 0)
+			(at 121.92 114.3 0)
 			(show_name yes)
 			(effects
@@
 		)
 		(property "HelpURL" "\\\\cern.ch\\dfs\\Applications\\Altium\\Datasheets\\MASW-008853.pdf"
-			(at 121.92 99.06 0)
+			(at 121.92 114.3 0)
 			(show_name yes)
 			(effects
@@
 		)
 		(property "ComponentLink1URL" ""
-			(at 121.92 99.06 0)
+			(at 121.92 114.3 0)
 			(show_name yes)
 			(effects
@@
 		)
 		(property "ComponentLink2URL" ""
-			(at 121.92 99.06 0)
+			(at 121.92 114.3 0)
 			(show_name yes)
 			(effects
@@
 		)
 		(property "ComponentLink2Description" ""
-			(at 121.92 99.06 0)
+			(at 121.92 114.3 0)
 			(show_name yes)
 			(effects
@@
 		)
 		(property "ComponentLink1Description" ""
-			(at 121.92 99.06 0)
+			(at 121.92 114.3 0)
 			(show_name yes)
 			(effects
@@
 		)
 		(property "CreateDate" "2025-07-10 00:00:00 +0000"
-			(at 121.92 99.06 0)
+			(at 121.92 114.3 0)
 			(show_name yes)
 			(effects
@@
 		)
 		(property "LatestRevisionDate" "2025-07-10 00:00:00 +0000"
-			(at 121.92 99.06 0)
+			(at 121.92 114.3 0)
 			(show_name yes)
 			(effects
@@
 		)
 		(property "SCEM" ""
-			(at 121.92 99.06 0)
+			(at 121.92 114.3 0)
 			(show_name yes)
 			(effects
@@
 		)
 		(property "LatestRevisionDate1" ""
-			(at 121.92 99.06 0)
+			(at 121.92 114.3 0)
 			(show_name yes)
 			(effects
@@
 		)
 		(property "Field1" ""
-			(at 121.92 99.06 0)
+			(at 121.92 114.3 0)
 			(show_name yes)
 			(effects
@@
 		)
 		(property "LibSymbol" "Analog & Interface:MASW-008853"
-			(at 121.92 99.06 0)
+			(at 121.92 114.3 0)
 			(show_name yes)
 			(effects
@@
 		)
 		(property "LibFootprint" "ICs And Semiconductors SMD:SOT65P210X110-6N"
-			(at 121.92 99.06 0)
+			(at 121.92 114.3 0)
 			(show_name yes)
 			(effects
@@
 		)
 		(property "Part Number" "MASW-008853"
-			(at 121.92 99.06 0)
+			(at 121.92 114.3 0)
 			(effects
 				(font
@@
 		)
 		(property "Database Name" "ICs And Semiconductors_Backup"
-			(at 121.92 99.06 0)
+			(at 121.92 114.3 0)
 			(effects
 				(font
@@
 		)
 		(property "Database Table Name" "Analog & Interface"
-			(at 121.92 99.06 0)
+			(at 121.92 114.3 0)
 			(effects
 				(font
@@
 		)
 		(property "Part Number Nocolon" "MASW-008853"
-			(at 121.92 99.06 0)
+			(at 121.92 114.3 0)
 			(effects
 				(font
@@
 	(symbol
 		(lib_id "power:GND")
-		(at 114.3 120.65 0)
+		(at 110.49 92.71 0)
 		(mirror y)
 		(unit 1)
@@
 		(dnp no)
 		(property "Reference" "#PWR0226"
-			(at 114.3 127 0)
+			(at 110.49 99.06 0)
 			(effects
 				(font
@@
 		)
 		(property "Value" "GND"
-			(at 114.3 124.46 0)
+			(at 110.49 96.52 0)
 			(effects
 				(font
@@
 		)
 		(property "Footprint" ""
-			(at 114.3 120.65 0)
+			(at 110.49 92.71 0)
 			(effects
 				(font
@@
 		)
 		(property "Datasheet" ""
-			(at 114.3 120.65 0)
+			(at 110.49 92.71 0)
 			(effects
 				(font
@@
 		)
 		(property "Description" "Power symbol creates a global label with name \"GND\" , ground"
-			(at 114.3 120.65 0)
+			(at 110.49 92.71 0)
 			(effects
 				(font

Commit message: Rerouted PCB Logic part
Parts:
- renumbered C131 to C1401, C132 to C1402, C133 to C1403, C134 to C1404, C135 to C1405, C136 to C1406, C137 to C1407, C138 to C1408, C139 to C1409, C140 to C1410, C141 to C1411, C142 to C1412, C143 to C1413, C144 to C1414, IC47 to IC1401, IC48 to IC1402, IC49 to IC1403, L24 to L1401, R83 to R1401, R84 to R1402, R85 to R1403, R86 to R1404, R87 to R1405, R88 to R1406, R89 to R1407, TR7 to TR1401
