File: DAC_AMPLIFIER_CH_A.kicad_sch (KiCad schematic)
At the start: 26 parts, among them IC1401 ${DEVICE}, IC1402 ${DEVICE}, IC1403 ${DEVICE}

Commit message: Routing new channels
Parts:
- renumbered C1401 to C1301, C1402 to C1302, C1403 to C1303, C1404 to C1304, C1405 to C1305, C1406 to C1306, C1407 to C1307, C1408 to C1308, C1409 to C1309, C1410 to C1310, C1411 to C1311, C1412 to C1312, C1413 to C1313, C1414 to C1314, IC1401 to IC1301, IC1402 to IC1302, IC1403 to IC1303, L1401 to L1301, R1401 to R1301, R1402 to R1302, R1403 to R1303, R1404 to R1304, R1405 to R1305, R1406 to R1306, R1407 to R1307, TR1401 to TR1301

Commit message: WIP snapshot
Parts:
- renumbered C1301 to C1401, C1302 to C1402, C1303 to C1403, C1304 to C1404, C1305 to C1405, C1306 to C1406, C1307 to C1407, C1308 to C1408, C1309 to C1409, C1310 to C1410, C1311 to C1411, C1312 to C1412, C1313 to C1413, C1314 to C1414, IC1301 to IC1401, IC1302 to IC1402, IC1303 to IC1403, L1301 to L1401, R1301 to R1401, R1302 to R1402, R1303 to R1403, R1304 to R1404, R1305 to R1405, R1306 to R1406, R1307 to R1407, TR1301 to TR1401

Commit message: Update project files and backups
Parts:
- added C1415, C1416: 1nF, Capacitors SMD:CAPC1005X55N, symbol CERN:Capacitors SMD/CC0402_1NF_50V_5%_C0G
Connections:
- net GND: now also C1415.2, C1416.2
- net OPAMP_BYPASS_V1_CH_A: now also C1415.1
- net OPAMP_BYPASS_V2_CH_A: now also C1416.1
