File: AFE_BLOCK_2.kicad_sch (KiCad schematic)
At the start: 2 parts, among them U2801 LPF, U2802 LPF

Commit message: Routing new channels
Parts:
- renumbered U2801 to U1201, U2802 to U1202
Changed lines of the file:
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@@
 		(dnp no)
 		(fields_autoplaced yes)
-		(property "Reference" "#PWR02802"
+		(property "Reference" "#PWR01202"
 			(at 59.69 140.97 0)
 			(effects
@@
 		(instances
 			(project "8CH_Analog_Front_END"
-				(path "/41597329-5145-432a-9041-5bc2cec82d9b/79457b0f-d794-4bf0-bdfc-49e38f4ce408"
-					(reference "#PWR02802")
+				(path "/41597329-5145-432a-9041-5bc2cec82d9b/e2455e95-2837-4323-b15c-07f24d19ff0e"
+					(reference "#PWR01202")
 					(unit 1)
 				)
@@
 		(dnp no)
 		(fields_autoplaced yes)
-		(property "Reference" "#PWR02801"
+		(property "Reference" "#PWR01201"
 			(at 59.69 113.03 0)
 			(effects
@@
 		(instances
 			(project "8CH_Analog_Front_END"
-				(path "/41597329-5145-432a-9041-5bc2cec82d9b/79457b0f-d794-4bf0-bdfc-49e38f4ce408"
-					(reference "#PWR02801")
+				(path "/41597329-5145-432a-9041-5bc2cec82d9b/e2455e95-2837-4323-b15c-07f24d19ff0e"
+					(reference "#PWR01201")
 					(unit 1)
 				)
@@
 		(dnp no)
 		(fields_autoplaced yes)
-		(property "Reference" "U2802"
+		(property "Reference" "U1202"
 			(at 45.085 111.76 0)
 			(effects
@@
 		(instances
 			(project "8CH_Analog_Front_END"
-				(path "/41597329-5145-432a-9041-5bc2cec82d9b/79457b0f-d794-4bf0-bdfc-49e38f4ce408"
-					(reference "U2802")
+				(path "/41597329-5145-432a-9041-5bc2cec82d9b/e2455e95-2837-4323-b15c-07f24d19ff0e"
+					(reference "U1202")
 					(unit 1)
 				)
@@
 		(dnp no)
 		(fields_autoplaced yes)
-		(property "Reference" "U2801"
+		(property "Reference" "U1201"
 			(at 45.085 83.82 0)
 			(effects
@@
 		(instances
 			(project "8CH_Analog_Front_END"
-				(path "/41597329-5145-432a-9041-5bc2cec82d9b/79457b0f-d794-4bf0-bdfc-49e38f4ce408"
-					(reference "U2801")
+				(path "/41597329-5145-432a-9041-5bc2cec82d9b/e2455e95-2837-4323-b15c-07f24d19ff0e"
+					(reference "U1201")
 					(unit 1)
 				)
@@
 		)
 		(instances
+			(project ""
+				(path "/e2455e95-2837-4323-b15c-07f24d19ff0e"
+					(page "#")
+				)
+			)
 			(project "8CH_Analog_Front_END"
-				(path "/41597329-5145-432a-9041-5bc2cec82d9b/79457b0f-d794-4bf0-bdfc-49e38f4ce408"
-					(page "38")
+				(path "/41597329-5145-432a-9041-5bc2cec82d9b/e2455e95-2837-4323-b15c-07f24d19ff0e"
+					(page "24")
 				)
 			)
@@
 		)
 		(instances
+			(project ""
+				(path "/e2455e95-2837-4323-b15c-07f24d19ff0e"
+					(page "#")
+				)
+			)
 			(project "8CH_Analog_Front_END"
-				(path "/41597329-5145-432a-9041-5bc2cec82d9b/79457b0f-d794-4bf0-bdfc-49e38f4ce408"
-					(page "29")
+				(path "/41597329-5145-432a-9041-5bc2cec82d9b/e2455e95-2837-4323-b15c-07f24d19ff0e"
+					(page "21")
 				)
 			)
@@
 		)
 		(instances
+			(project ""
+				(path "/e2455e95-2837-4323-b15c-07f24d19ff0e"
+					(page "#")
+				)
+			)
 			(project "8CH_Analog_Front_END"
-				(path "/41597329-5145-432a-9041-5bc2cec82d9b/79457b0f-d794-4bf0-bdfc-49e38f4ce408"
-					(page "34")
+				(path "/41597329-5145-432a-9041-5bc2cec82d9b/e2455e95-2837-4323-b15c-07f24d19ff0e"
+					(page "13")
 				)
 			)
@@
 		)
 		(instances
+			(project ""
+				(path "/e2455e95-2837-4323-b15c-07f24d19ff0e"
+					(page "#")
+				)
+			)
 			(project "8CH_Analog_Front_END"
-				(path "/41597329-5145-432a-9041-5bc2cec82d9b/79457b0f-d794-4bf0-bdfc-49e38f4ce408"
-					(page "30")
+				(path "/41597329-5145-432a-9041-5bc2cec82d9b/e2455e95-2837-4323-b15c-07f24d19ff0e"
+					(page "23")
 				)
 			)
@@
 		)
 		(instances
+			(project ""
+				(path "/e2455e95-2837-4323-b15c-07f24d19ff0e"
+					(page "#")
+				)
+			)
 			(project "8CH_Analog_Front_END"
-				(path "/41597329-5145-432a-9041-5bc2cec82d9b/79457b0f-d794-4bf0-bdfc-49e38f4ce408"
-					(page "35")
+				(path "/41597329-5145-432a-9041-5bc2cec82d9b/e2455e95-2837-4323-b15c-07f24d19ff0e"
+					(page "20")
 				)
 			)
@@
 		)
 		(instances
+			(project ""
+				(path "/e2455e95-2837-4323-b15c-07f24d19ff0e"
+					(page "#")
+				)
+			)
 			(project "8CH_Analog_Front_END"
-				(path "/41597329-5145-432a-9041-5bc2cec82d9b/79457b0f-d794-4bf0-bdfc-49e38f4ce408"
-					(page "31")
+				(path "/41597329-5145-432a-9041-5bc2cec82d9b/e2455e95-2837-4323-b15c-07f24d19ff0e"
+					(page "25")
 				)
 			)
@@
 		)
 		(instances
+			(project ""
+				(path "/e2455e95-2837-4323-b15c-07f24d19ff0e"
+					(page "#")
+				)
+			)
 			(project "8CH_Analog_Front_END"
-				(path "/41597329-5145-432a-9041-5bc2cec82d9b/79457b0f-d794-4bf0-bdfc-49e38f4ce408"
-					(page "32")
+				(path "/41597329-5145-432a-9041-5bc2cec82d9b/e2455e95-2837-4323-b15c-07f24d19ff0e"
+					(page "22")
 				)
 			)
@@
 		)
 		(instances
+			(project ""
+				(path "/e2455e95-2837-4323-b15c-07f24d19ff0e"
+					(page "#")
+				)
+			)
 			(project "8CH_Analog_Front_END"
-				(path "/41597329-5145-432a-9041-5bc2cec82d9b/79457b0f-d794-4bf0-bdfc-49e38f4ce408"
-					(page "36")
+				(path "/41597329-5145-432a-9041-5bc2cec82d9b/e2455e95-2837-4323-b15c-07f24d19ff0e"
+					(page "18")
 				)
 			)
@@
 		)
 		(instances
+			(project ""
+				(path "/e2455e95-2837-4323-b15c-07f24d19ff0e"
+					(page "#")
+				)
+			)
 			(project "8CH_Analog_Front_END"
-				(path "/41597329-5145-432a-9041-5bc2cec82d9b/79457b0f-d794-4bf0-bdfc-49e38f4ce408"
-					(page "33")
+				(path "/41597329-5145-432a-9041-5bc2cec82d9b/e2455e95-2837-4323-b15c-07f24d19ff0e"
+					(page "26")
 				)
 			)
@@
 		)
 		(instances
+			(project ""
+				(path "/e2455e95-2837-4323-b15c-07f24d19ff0e"
+					(page "#")
+				)
+			)
 			(project "8CH_Analog_Front_END"
-				(path "/41597329-5145-432a-9041-5bc2cec82d9b/79457b0f-d794-4bf0-bdfc-49e38f4ce408"
-					(page "37")
-				)
-			)
+				(path "/41597329-5145-432a-9041-5bc2cec82d9b/e2455e95-2837-4323-b15c-07f24d19ff0e"
+					(page "19")
+				)
+			)
