File: 8CH_Analog_Front_END.kicad_sch (KiCad schematic)
At the start: 0 parts

Commit message: Routing finished
Other:
- added sheet MECHANICAL (MECHANICAL.kicad_sch)

Commit message: WIP snapshot
Parts:
- added R101, R103, R104, R105: 220, Resistors SMD:RESC1005X40N, symbol CERN:Resistors SMD/R0402_220R_1%_0.0625W_100PPM
- added R102: 4k7, Resistors SMD:RESC1005X40N, symbol CERN_Linux:Resistors SMD/R0402_4K7_1%_0.0625W_100PPM
Connections:
- net SER_CLK: now also R105.2
- new net +3V3D: R102.2
- new net B84_RFU0: R103.2
- new net B84_RFU1: R101.2
- new net GND: R101.1, R103.1, R104.1, R105.1
- new net SER_RCLK: R104.2
Other:
- removed sheet MUX
- removed sheet RFSoC_Connector_X1
- added sheet ADC_DAC_Clock_Synthesizer (ADC_DAC_Clock_Synthesizer.kicad_sch)
- added sheet RFSoC_Connector_X2 (RFSoC_Connector_X1.kicad_sch)
- sheet AFE_BLOCK_0 ports: added SER_DATA_IN_A, SER_DATA_IN_B, SER_RCLK, SER_RST_N; removed D_LATCH_OE, SER_DATA, SER_LATCH_CH_A, SER_LATCH_CH_B
- sheet AFE_BLOCK_1: file AFE_BLOCK_1.kicad_sch -> AFE_BLOCK.kicad_sch
- sheet AFE_BLOCK_1 ports: added SER_DATA_IN_A, SER_DATA_IN_B, SER_RCLK, SER_RST_N; removed D_LATCH_OE, SER_DATA, SER_LATCH_CH_A, SER_LATCH_CH_B
- sheet AFE_BLOCK_2: file AFE_BLOCK_2.kicad_sch -> AFE_BLOCK.kicad_sch
- sheet AFE_BLOCK_2 ports: added SER_DATA_IN_A, SER_DATA_IN_B, SER_RCLK, SER_RST_N; removed D_LATCH_OE, SER_DATA, SER_LATCH_CH_A, SER_LATCH_CH_B
- sheet AFE_BLOCK_3: file AFE_BLOCK_3.kicad_sch -> AFE_BLOCK.kicad_sch
- sheet AFE_BLOCK_3 ports: added SER_DATA_IN_A, SER_DATA_IN_B, SER_RCLK, SER_RST_N; removed D_LATCH_OE, SER_DATA, SER_LATCH_CH_A, SER_LATCH_CH_B
- sheet DATA_BUFFER ports: added SER_CLK_CH[0..3], SER_DATA[0..7], SER_DATA_FPGA[0..7], SER_RCLK_CH[0..3], SER_RCLK_FPGA; removed D_LATCH_OE, D_LATCH_OE_FPGA, SER_CLK, SER_DATA, SER_DATA_FPGA
- note added: "Fixme: Add your digital connections acordingly and did not know how many resistors you want for debuging"
- note added: "Optional parallel termination resistors for shifreg clock lines. Left just in case we had excessive ringing :-)"
- note added: "Two digital 3.3V lines for future use, the dummy resistors are just placeholders for easy rework."
- note removed: "MUX Toggle Pin Out MUX Addr S0 Pin Out MUX Addr S2 Pin Out MUX Addr S1 Pin Out"
- note removed: "Serial DATA Serial CLOCK Serial D_LATCH"

Commit message: Update project files and backups
Parts:
- removed R102: 4k7, Resistors SMD:RESC1005X40N, symbol CERN_Linux:Resistors SMD/R0402_4K7_1%_0.0625W_100PPM
- removed R104: 220, Resistors SMD:RESC1005X40N, symbol CERN:Resistors SMD/R0402_220R_1%_0.0625W_100PPM
- added R102, R104: 100, Resistors SMD:RESC1005X40N, symbol CERN_Linux:Resistors SMD/R0402_100R_1%_0.1W_100PPM
Connections:
- net ADC_DAC_Clock_Synthesizer/CLK_SPI_SCK: now also R104.1
- net ADC_DAC_Clock_Synthesizer/CLK_SPI_SDI: now also R102.1
- net SER_CLK renamed B84_RFU2
- new net RFSoC_Connector_X2/B84.L10N_D19_AV7: R102.2
- new net RFSoC_Connector_X2/B84.L11N_D21_AR6: R104.2
- no-connect marks 0 -> 4
Other:
- note added: "Flipped for easier routing"
- note added: "Three digital 3.3V lines for future use, the dummy resistors are just placeholders for easy rework."
- note removed: "Optional parallel termination resistors for shifreg clock lines. Left just in case we had excessive ringing :-)"
- note removed: "Two digital 3.3V lines for future use, the dummy resistors are just placeholders for easy rework."
