File: ADC_DAC_Clock_Synthesizer.kicad_sch (KiCad schematic)
At the start: 10 parts

Commit message: Update project files and backups
Parts:
- added C403, C404: 1nF, Capacitors SMD:CAPC1005X55N, symbol CERN:Capacitors SMD/CC0402_1NF_50V_5%_C0G
Connections:
- net +1V2_CLK_BIAS: now also C403.2, C404.2
- net GND: now also C403.1, C404.1
