File: CHANNEL_LOGIC_CONTROL.kicad_sch (KiCad schematic)
At the start: 63 parts, among them IC1601 ${DEVICE}, IC1602 ${DEVICE}, IC1603 ${DEVICE}, IC1604 ${DEVICE}, IC1605 ${DEVICE}, IC1606 ${DEVICE}

Commit message: Update project files and backups
Parts:
- removed C1601, C1602, C1603, C1604, C1605, C1606, C1607, C1608, C1609: 100nF, Capacitors SMD:CAPC1608X87N, symbol CERN:Capacitors SMD/CC0603_100NF_50V_10%_X7R
- removed C1633: 1nF, Capacitors SMD:CAPC1005X55N, symbol CERN:Capacitors SMD/CC0402_1NF_50V_5%_C0G
- removed R1624: 22R6, Resistors SMD:RESC1005X40N, symbol CERN:Resistors SMD/R0402_22R6_1%_0.063W_100PPM
- added C1, C17, C18, C33, C34, C49, C73, C81, C9: 100nF, Capacitors SMD:CAPC1005X55N, symbol CERN:Capacitors SMD/CC0402_100NF_50V_10%_X7R
Connections:
- net +3V3D: now also C1.2, C17.2, C33.2, C34.2, C49.2, C73.2, C81.2
- net +5VD: now also C18.2, C9.2
- net GND: now also C1.1, C17.1, C18.1, C33.1, C34.1, C49.1, C73.1, C81.1, C9.1
- net IO_5V_2: now reaches C1612.1, R1607.2
- net IO_5V_15: now reaches C1625.1, R1623.2
- net IO_5V_14: now reaches C1624.1, R1620.2
- net IO_5V_3: now reaches C1613.1, R1610.2
- net 1BITTTEN_VC1_CH renamed IO_5V_12
- net 1BITTTEN_VC2_CH renamed IO_5V_13
- net A0 renamed IO_3V3_0
- net A1 renamed IO_3V3_1
- net A2 renamed IO_3V3_2
- net A3 renamed IO_3V3_3
- net A4 renamed IO_3V3_4
- net A5 renamed IO_3V3_5
- net A6 renamed IO_3V3_6
- net C1_1dB renamed IO_5V_8
- net C2_2dB renamed IO_5V_9
- net C4_4dB renamed IO_5V_10
- net C8_8dB renamed IO_5V_11
- net CAL_MEAS_SW_VC1_CH renamed IO_5V_0
- net CAL_MEAS_SW_VC2_CH renamed IO_5V_1
- net DAC_DIR_V1_CH renamed IO_5V_7
- net DAC_DIR_V2_CH renamed IO_5V_6
- net OPAMP_BYPASS_V1_CH renamed IO_5V_4
- net OPAMP_BYPASS_V2_CH renamed IO_5V_5
- no-connect marks 1 -> 2
