File: DAC_AMPLIFIER_CH_B.kicad_sch (KiCad schematic)
At the start: 26 parts, among them IC1501 ${DEVICE}, IC1502 ${DEVICE}, IC1503 ${DEVICE}

Commit message: WIP snapshot
Parts:
- renumbered C1501 to C1301, C1502 to C1302, C1503 to C1303, C1504 to C1304, C1505 to C1305, C1506 to C1306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
