File: Master_Clock_Generator.kicad_sch (KiCad schematic)
At the start: 68 parts, among them IC201 ${DEVICE}, IC202 ${DEVICE}, IC203 ${DEVICE}, J201 125M out

Commit message: Update project files and backups
Parts:
- removed R211, R212: 100, Resistors SMD:RESC1005X40N, symbol CERN_Linux:Resistors SMD/R0402_100R_1%_0.1W_100PPM
Connections:
- net SPI_MOSI: now also IC203.18 (SDA/SDIO)
- net SPI_SCK: now also IC203.16 (SCLK)
- net SYSCLOCK_62M5_1V2_N: now also C238.1; no longer C242.1
- net SYSCLOCK_62M5_1V2_P: now also C242.1; no longer C238.1
- net SYSREF_7M_1V2_N: now also C240.1; no longer C244.1
- net SYSREF_7M_1V2_P: now also C244.1; no longer C240.1
