File: RF_5GHz_PLL.kicad_sch (KiCad schematic)
At the start: 83 parts, among them IC5201 ${DEVICE}, IC5202 ${DEVICE}, J5201 5G out

Commit message: Update project files and backups
Parts:
- removed R5205, R5206: 100, Resistors SMD:RESC1005X40N, symbol CERN_Linux:Resistors SMD/R0402_100R_1%_0.1W_100PPM
Connections:
- net CLK_A_5G_N: now also C5254.2; no longer C5255.2
- net CLK_A_5G_P: now also C5255.2; no longer C5254.2
- net CLK_B_5G_N: now also C5256.2; no longer C5257.2
- net CLK_B_5G_P: now also C5257.2; no longer C5256.2
- net LMX_SCK: now also IC5202.16 (SCK)
- net LMX_SDI: now also IC5202.17 (SDI)
Other:
- note added: "Both clocks inverted for ease of routing"
