File: RF_SWITCH_CONTROL.kicad_sch (KiCad schematic)
At the start: 12 parts, among them IC1 ${DEVICE}, IC2 ${DEVICE}

Commit message: Rerouted PCB Logic part
Parts:
- renumbered C1 to C2701, IC1 to IC2701, IC2 to IC2702, L1 to L2701, R1 to R2701, R2 to R2702, R3 to R2703, R14 to R2704, R13 to R2705, R11 to R2706, R12 to R2707, R15 to R2708
Changed lines of the file:
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@@
 		(dnp no)
 		(fields_autoplaced yes)
-		(property "Reference" "IC2"
+		(property "Reference" "IC2702"
 			(at 182.88 68.58 0)
 			(effects
@@
 			(project ""
 				(path "/41597329-5145-432a-9041-5bc2cec82d9b/e1bc8eb5-1b45-4220-9961-d777b4d01cb8"
-					(reference "IC2")
+					(reference "IC2702")
 					(unit 2)
 				)
@@
 		(on_board yes)
 		(dnp no)
-		(property "Reference" "R13"
+		(property "Reference" "R2705"
 			(at 189.23 35.052 0)
 			(effects
@@
 			(project "8CH_Analog_Front_END"
 				(path "/41597329-5145-432a-9041-5bc2cec82d9b/e1bc8eb5-1b45-4220-9961-d777b4d01cb8"
-					(reference "R13")
+					(reference "R2705")
 					(unit 1)
 				)
@@
 		(dnp no)
 		(fields_autoplaced yes)
-		(property "Reference" "#PWR03"
+		(property "Reference" "#PWR02707"
 			(at 195.58 151.13 0)
 			(effects
@@
 			(project "8CH_Analog_Front_END"
 				(path "/41597329-5145-432a-9041-5bc2cec82d9b/e1bc8eb5-1b45-4220-9961-d777b4d01cb8"
-					(reference "#PWR03")
+					(reference "#PWR02707")
 					(unit 1)
 				)
@@
 		(on_board yes)
 		(dnp no)
-		(property "Reference" "R11"
+		(property "Reference" "R2706"
 			(at 189.23 62.992 0)
 			(effects
@@
 			(project "8CH_Analog_Front_END"
 				(path "/41597329-5145-432a-9041-5bc2cec82d9b/e1bc8eb5-1b45-4220-9961-d777b4d01cb8"
-					(reference "R11")
+					(reference "R2706")
 					(unit 1)
 				)
@@
 		(dnp no)
 		(fields_autoplaced yes)
-		(property "Reference" "#PWR04"
+		(property "Reference" "#PWR02703"
 			(at 90.17 31.75 0)
 			(effects
@@
 			(project "8CH_Analog_Front_END"
 				(path "/41597329-5145-432a-9041-5bc2cec82d9b/e1bc8eb5-1b45-4220-9961-d777b4d01cb8"
-					(reference "#PWR04")
+					(reference "#PWR02703")
 					(unit 1)
 				)
@@
 		(dnp no)
 		(fields_autoplaced yes)
-		(property "Reference" "#PWR08"
+		(property "Reference" "#PWR02705"
 			(at 124.46 85.09 0)
 			(effects
@@
 			(project "8CH_Analog_Front_END"
 				(path "/41597329-5145-432a-9041-5bc2cec82d9b/e1bc8eb5-1b45-4220-9961-d777b4d01cb8"
-					(reference "#PWR08")
+					(reference "#PWR02705")
 					(unit 1)
 				)
@@
 		(dnp no)
 		(fields_autoplaced yes)
-		(property "Reference" "IC2"
+		(property "Reference" "IC2702"
 			(at 182.88 124.46 0)
 			(effects
@@
 			(project ""
 				(path "/41597329-5145-432a-9041-5bc2cec82d9b/e1bc8eb5-1b45-4220-9961-d777b4d01cb8"
-					(reference "IC2")
+					(reference "IC2702")
 					(unit 4)
 				)
@@
 		(on_board yes)
 		(dnp no)
-		(property "Reference" "L1"
+		(property "Reference" "L2701"
 			(at 77.47 76.962 0)
 			(effects
@@
 			(project "8CH_Analog_Front_END"
 				(path "/41597329-5145-432a-9041-5bc2cec82d9b/e1bc8eb5-1b45-4220-9961-d777b4d01cb8"
-					(reference "L1")
+					(reference "L2701")
 					(unit 1)
 				)
@@
 		(on_board yes)
 		(dnp no)
-		(property "Reference" "IC1"
+		(property "Reference" "IC2701"
 			(at 111.76 25.4 0)
 			(effects
@@
 			(project "8CH_Analog_Front_END"
 				(path "/41597329-5145-432a-9041-5bc2cec82d9b/e1bc8eb5-1b45-4220-9961-d777b4d01cb8"
-					(reference "IC1")
+					(reference "IC2701")
 					(unit 1)
 				)
@@
 		(dnp no)
 		(fields_autoplaced yes)
-		(property "Reference" "IC2"
+		(property "Reference" "IC2702"
 			(at 182.88 40.64 0)
 			(effects
@@
 			(project ""
 				(path "/41597329-5145-432a-9041-5bc2cec82d9b/e1bc8eb5-1b45-4220-9961-d777b4d01cb8"
-					(reference "IC2")
+					(reference "IC2702")
 					(unit 1)
 				)
@@
 		(on_board yes)
 		(dnp no)
-		(property "Reference" "R12"
+		(property "Reference" "R2707"
 			(at 189.23 90.932 0)
 			(effects
@@
 			(project "8CH_Analog_Front_END"
 				(path "/41597329-5145-432a-9041-5bc2cec82d9b/e1bc8eb5-1b45-4220-9961-d777b4d01cb8"
-					(reference "R12")
+					(reference "R2707")
 					(unit 1)
 				)
@@
 		(dnp no)
 		(fields_autoplaced yes)
-		(property "Reference" "#PWR05"
+		(property "Reference" "#PWR02704"
 			(at 90.17 104.14 0)
 			(effects
@@
 			(project "8CH_Analog_Front_END"
 				(path "/41597329-5145-432a-9041-5bc2cec82d9b/e1bc8eb5-1b45-4220-9961-d777b4d01cb8"
-					(reference "#PWR05")
+					(reference "#PWR02704")
 					(unit 1)
 				)
@@
 		(on_board yes)
 		(dnp no)
-		(property "Reference" "C1"
+		(property "Reference" "C2701"
 			(at 87.122 85.09 0)
 			(effects
@@
 			(project "8CH_Analog_Front_END"
 				(path "/41597329-5145-432a-9041-5bc2cec82d9b/e1bc8eb5-1b45-4220-9961-d777b4d01cb8"
-					(reference "C1")
+					(reference "C2701")
 					(unit 1)
 				)
@@
 		(on_board yes)
 		(dnp no)
-		(property "Reference" "R15"
+		(property "Reference" "R2708"
 			(at 189.23 118.872 0)
 			(effects
@@
 			(project "8CH_Analog_Front_END"
 				(path "/41597329-5145-432a-9041-5bc2cec82d9b/e1bc8eb5-1b45-4220-9961-d777b4d01cb8"
-					(reference "R15")
+					(reference "R2708")
 					(unit 1)
 				)
@@
 		(dnp no)
 		(fields_autoplaced yes)
-		(property "Reference" "IC2"
+		(property "Reference" "IC2702"
 			(at 182.88 96.52 0)
 			(effects
@@
 			(project ""
 				(path "/41597329-5145-432a-9041-5bc2cec82d9b/e1bc8eb5-1b45-4220-9961-d777b4d01cb8"
-					(reference "IC2")
+					(reference "IC2702")
 					(unit 3)
 				)
@@
 		(on_board yes)
 		(dnp yes)
-		(property "Reference" "R14"
+		(property "Reference" "R2704"
 			(at 55.372 68.58 0)
 			(effects
@@
 			(project "8CH_Analog_Front_END"
 				(path "/41597329-5145-432a-9041-5bc2cec82d9b/e1bc8eb5-1b45-4220-9961-d777b4d01cb8"
-					(reference "R14")
+					(reference "R2704")
 					(unit 1)
 				)
@@
 		(on_board yes)
 		(dnp yes)
-		(property "Reference" "R3"
+		(property "Reference" "R2703"
 			(at 49.022 68.58 0)
 			(effects
@@
 			(project "8CH_Analog_Front_END"
 				(path "/41597329-5145-432a-9041-5bc2cec82d9b/e1bc8eb5-1b45-4220-9961-d777b4d01cb8"
-					(reference "R3")
+					(reference "R2703")
 					(unit 1)
 				)
@@
 		(dnp no)
 		(fields_autoplaced yes)
-		(property "Reference" "#PWR01"
+		(property "Reference" "#PWR02701"
 			(at 44.45 85.09 0)
 			(effects
@@
 			(project "8CH_Analog_Front_END"
 				(path "/41597329-5145-432a-9041-5bc2cec82d9b/e1bc8eb5-1b45-4220-9961-d777b4d01cb8"
-					(reference "#PWR01")
+					(reference "#PWR02701")
 					(unit 1)
 				)
@@
 		(on_board yes)
 		(dnp yes)
-		(property "Reference" "R2"
+		(property "Reference" "R2702"
 			(at 42.672 68.58 0)
 			(effects
@@
 			(project "8CH_Analog_Front_END"
 				(path "/41597329-5145-432a-9041-5bc2cec82d9b/e1bc8eb5-1b45-4220-9961-d777b4d01cb8"
-					(reference "R2")
+					(reference "R2702")
 					(unit 1)
 				)
@@
 		(dnp no)
 		(fields_autoplaced yes)
-		(property "Reference" "#PWR02"
+		(property "Reference" "#PWR02702"
 			(at 66.04 78.74 0)
 			(effects
@@
 			(project "8CH_Analog_Front_END"
 				(path "/41597329-5145-432a-9041-5bc2cec82d9b/e1bc8eb5-1b45-4220-9961-d777b4d01cb8"
-					(reference "#PWR02")
+					(reference "#PWR02702")
 					(unit 1)
 				)
@@
 		(on_board yes)
 		(dnp yes)
-		(property "Reference" "R1"
+		(property "Reference" "R2701"
 			(at 36.322 68.58 0)
 			(effects
@@
 			(project "8CH_Analog_Front_END"
 				(path "/41597329-5145-432a-9041-5bc2cec82d9b/e1bc8eb5-1b45-4220-9961-d777b4d01cb8"
-					(reference "R1")
+					(reference "R2701")
 					(unit 1)
 				)
@@
 		(dnp no)
 		(fields_autoplaced yes)
-		(property "Reference" "#PWR09"
+		(property "Reference" "#PWR02706"
 			(at 165.1 147.32 0)
 			(effects
@@
 			(project "8CH_Analog_Front_END"
 				(path "/41597329-5145-432a-9041-5bc2cec82d9b/e1bc8eb5-1b45-4220-9961-d777b4d01cb8"
-					(reference "#PWR09")
+					(reference "#PWR02706")
 					(unit 1)
 				)

Commit message: Routing the Power Sector
Parts:
- added C2702: 100nF, Capacitors SMD:CAPC1005X55N, symbol CERN:Capacitors SMD/CC0402_100NF_25V_10%_X7R_YUDEN_TMK105B7104KVHF
- added L2702: 220R@100MHz, Inductors SMD:INDC1608X95N, symbol CERN:Inductors SMD/IND0603_MURATA_BLM18SG221TN1 [alt]
Connections:
- net +5VD: now also L2702.2; no longer IC2702.14 (VCC)
- net GND: now also C2702.1
- new net: C2702.2, IC2702.14 (VCC), L2702.1

Commit message: WIP snapshot
Parts:
- removed R2701, R2702, R2703, R2704: 0, Resistors SMD:RESC1005X40N, symbol CERN:Resistors SMD/R0402_0R_JUMPER
- added C2701, C2702: 100nF, Capacitors SMD:CAPC1608X87N, symbol CERN:Capacitors SMD/CC0603_100NF_50V_10%_X7R
- added IC2701: ${DEVICE}, ICs And Semiconductors SMD:TEXAS_RHL (S-PVQFN-N24), symbol CERN_Linux:Standard Logic/SN74LVC8T245RHL
- added R2701, R2702, R2703, R2704: 4k7, Resistors SMD:RESC1005X40N, symbol CERN_Linux:Resistors SMD/R0402_4K7_1%_0.0625W_100PPM
- renumbered C2701 to C2703, C2702 to C2704, IC2701 to IC2702, IC2702 to IC2703
Connections:
- net GND: now also C2701.1, C2702.1, IC2701.10 (A8), IC2701.11 (GND), IC2701.12 (GND), IC2701.13 (GND), IC2701.22 (~{OE}), IC2701.7 (A5), IC2701.8 (A6), IC2701.9 (A7), R2701.2, R2702.2, R2703.2, R2704.2
- net RF_SW_0: now also IC2701.3 (A1), R2704.1; no longer IC2702.2 (1A), IC2702.3 (2A)
- net RF_SW_1: now also IC2701.4 (A2), R2703.1; no longer IC2702.4 (3A), IC2702.5 (4A)
- net RF_SW_2: now also IC2701.5 (A3), R2702.1; no longer IC2702.6 (5A), IC2702.7 (6A)
- net RF_SW_3: now also IC2701.6 (A4), R2701.1; no longer IC2702.8 (7A), IC2702.9 (8A)
- net at IC2703.12 (B), IC2703.13 (A): no longer IC2702.11 (8Y)
- new net: IC2701.18 (B4), IC2702.8 (7A), IC2702.9 (8A)
- new net: IC2701.19 (B3), IC2702.6 (5A), IC2702.7 (6A)
- new net: IC2701.20 (B2), IC2702.4 (3A), IC2702.5 (4A)
- new net: IC2701.21 (B1), IC2702.2 (1A), IC2702.3 (2A)
- new net +3V3D: C2701.2, C2702.2, IC2701.1 (VCCA), IC2701.2 (DIR), IC2701.23 (VCCB), IC2701.24 (VCCB)
- no-connect marks 0 -> 4
Other:
- note added: "3.3V buffer "just in case". I wouldn't like an accidental +5V frying the SoM."
- moved on the sheet: C2703, C2704, IC2702, IC2703A, IC2703B, IC2703C, IC2703D, L2701, L2702, R2705, R2706, R2707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

Commit message: Update project files and backups
Parts:
- removed C2701, C2702: 100nF, Capacitors SMD:CAPC1608X87N, symbol CERN:Capacitors SMD/CC0603_100NF_50V_10%_X7R
- removed R2705, R2706, R2707, R2708: 0, Resistors SMD:RESC1005X40N, symbol CERN:Resistors SMD/R0402_0R_JUMPER
- added C2701, C2702: 100nF, Capacitors SMD:CAPC1005X55N, symbol CERN:Capacitors SMD/CC0402_100NF_25V_10%_X7R_YUDEN_TMK105B7104KVHF
- added R2705, R2706, R2707, R2708, R2709, R2710, R2711, R2712: 22R6, Resistors SMD:RESC1005X40N, symbol CERN:Resistors SMD/R0402_22R6_1%_0.063W_100PPM
Connections:
- net +3V3D: now also C2701.2, C2702.2
- net GND: now also C2701.1, C2702.1
- net RF_SW_VC1_CH_0: now also R2705.2
- net RF_SW_VC1_CH_1: now also R2706.2
- net RF_SW_VC1_CH_2: now also R2707.2
- net RF_SW_VC1_CH_3: now also R2708.2
- net RF_SW_VC2_CH_0: now also R2709.1; no longer IC2703.3 (~{O})
- net RF_SW_VC2_CH_1: now also R2710.2; no longer IC2703.6 (~{O})
- net RF_SW_VC2_CH_2: now also R2711.2; no longer IC2703.8 (~{O})
- net RF_SW_VC2_CH_3: now also R2712.2; no longer IC2703.11 (~{O})
- net at IC2702.18 (1Y): now also R2705.1
- net at IC2702.16 (3Y): now also R2706.1
- net at IC2703.12 (B), IC2703.13 (A): now also IC2702.11 (8Y)
- net at IC2702.12 (7Y): now also R2708.1
- net at IC2702.14 (5Y): now also R2707.1
- new net: IC2703.6 (~{O}), R2710.1
- new net: IC2703.11 (~{O}), R2712.1
- new net: IC2703.3 (~{O}), R2709.2
- new net: IC2703.8 (~{O}), R2711.1
