File: SWITCH_CONTROLL.kicad_sch (KiCad schematic)
At the start: 17 parts, among them IC1101 ${DEVICE}, IC1102 ${DEVICE}, IC1103 ${DEVICE}, IC1104 ${DEVICE}, IC1105 ${DEVICE}

Commit message: WIP snapshot
Parts:
- removed C1101, C1102, C1103, C1105, C1107, C1108, C1109, C1110, C1111, C1112: 10nF, Capacitors SMD:CAPC1005X55N, symbol CERN:Capacitors SMD/CC0402_10NF_50V_5%_X7R
- added C1101, C1102, C1105, C1106, C1107, C1108, C1109, C1110: 100nF, Capacitors SMD:CAPC1005X55N, symbol CERN:Capacitors SMD/CC0402_100NF_50V_10%_X7R
- renumbered C1104 to C1103, C1106 to C1104
Connections:
- net CH_A: now also C1107.1
- net CH_B: now also C1108.1
- net SW_CROSS_BAR_OUT_CH_A: now also C1109.2
- net SW_CROSS_BAR_OUT_CH_B: now also C1110.2
- net SW_DAC_CALL_IN_CH_A: now also IC1101.5 (RFC)
- net SW_DAC_CALL_IN_CH_B: now also IC1104.5 (RFC)
- net at IC1101.3 (RF2): now also C1105.1
- net at IC1102.12 (TX): now also C1105.2
- net at IC1105.6 (ANT2): now also C1108.2
- net at IC1101.1 (RF1): now also C1101.2
- net at IC1102.4 (ANT1): now also C1101.1
- net at IC1104.3 (RF2): now also C1102.2
- net at IC1103.12 (TX): now also C1102.1
- net at IC1105.4 (ANT1): now also C1107.2
- net at IC1105.10 (RX): now also C1110.1
- net at IC1105.12 (TX): now also C1109.1
- net at IC1104.1 (RF1): now also C1106.1
- net at IC1103.4 (ANT1): now also C1106.2

Commit message: Update project files and backups
Parts:
- added C1111, C1112: 1nF, Capacitors SMD:CAPC1005X55N, symbol CERN:Capacitors SMD/CC0402_1NF_50V_5%_C0G
Connections:
- net GND: now also C1111.1, C1112.1
- net VC1_RF_SW_CONTROL: now also C1111.2
- net VC2_RF_SW_CONTROL: now also C1112.2
